File: samd51_wroom.brd (EAGLE design)
At the start: 25.5 x 18 mm, 19 parts, among them X5 32.768

Commit message: mk1 fabbed
Parts:
- removed U$15: AMPHENOL_MICRO_USB, 00_bsiepert:AMPHENOL_MICRO_USB
- added U$19: AMPHENOL_MICRO_USBAMPHENOL_MICRO_USB_BETTER, 00_bsiepert:BETTER_AMP_MICRO_USB
Connections:
- removed net N$4: U$1.41
- net GND: now also U$19.GND; no longer U$15.P$5
- net USB+: now also U$19.USB_P; no longer U$15.P$3
- net USB-: now also U$19.USB_N; no longer U$15.P$2
- net VDDCORE: now also U$1.41
Routing:
- net GND: track 11.4 -> 13.8 mm
- net VDDCORE: track 5.74 -> 6.61 mm
