File: samd51_wroom.sch (EAGLE design)
At the start: 19 parts, among them X5 32.768

Commit message: added SWD and USB headers  :|
Parts:
- added U$15: AMPHENOL_MICRO_USB, 00_bsiepert:AMPHENOL_MICRO_USB
- added X2: 2x5 0.05" SWD, microbuilder:JTAG-CORTEXBOXPOSTS
Connections:
- net GND: now also X2.GND@1, X2.GND@2
- net RESET_SW: now also X2.NRESET
- net SWCLK: now also X2.SWDCLK
- net SWDIO: now also X2.SWDIO
- net VDDIO: now also X2.VCC
Other:
- moved on the sheet: TP1, TP2
Changed lines of the file:
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@@
 <part name="U$14" library="microbuilder" deviceset="GND" device=""/>
 <part name="R2" library="microbuilder" deviceset="RESISTOR" device="_0603_NOOUT" value="330"/>
+<part name="X2" library="microbuilder" deviceset="JTAG-CORTEX" device="BOXPOSTS" value="2x5 0.05&quot; SWD"/>
+<part name="U$15" library="00_bsiepert" deviceset="AMPHENOL_MICRO_USB" device=""/>
 </parts>
 <sheets>
@@
 <instance part="U$12" gate="G$1" x="304.8" y="-12.7"/>
 <instance part="U$13" gate="G$1" x="134.62" y="-12.7"/>
-<instance part="TP1" gate="G$1" x="416.56" y="121.92"/>
-<instance part="TP2" gate="G$1" x="416.56" y="119.38"/>
+<instance part="TP1" gate="G$1" x="403.86" y="149.86" rot="R90"/>
+<instance part="TP2" gate="G$1" x="406.4" y="149.86" rot="R90"/>
 <instance part="C1" gate="G$1" x="335.28" y="121.92"/>
 <instance part="U$14" gate="G$1" x="335.28" y="132.08" rot="R180"/>
 <instance part="R2" gate="G$1" x="340.36" y="139.7" rot="MR90"/>
+<instance part="X2" gate="G$1" x="416.56" y="142.24" rot="MR0"/>
+<instance part="U$15" gate="G$1" x="337.82" y="182.88" rot="R180"/>
 </instances>
 <busses>
@@
 <pinref part="U$14" gate="G$1" pin="GND"/>
 </segment>
+<segment>
+<pinref part="X2" gate="G$1" pin="GND@1"/>
+<wire x1="424.18" y1="144.78" x2="426.72" y2="144.78" width="0.1524" layer="91"/>
+<wire x1="426.72" y1="144.78" x2="426.72" y2="142.24" width="0.1524" layer="91"/>
+<pinref part="X2" gate="G$1" pin="GND@2"/>
+<wire x1="426.72" y1="142.24" x2="424.18" y2="142.24" width="0.1524" layer="91"/>
+<label x="426.72" y="142.24" size="1.778" layer="95"/>
+</segment>
 </net>
 <net name="!RESET" class="0">
@@
 <wire x1="322.58" y1="111.76" x2="304.8" y2="129.54" width="0.1524" layer="91"/>
 <wire x1="304.8" y1="129.54" x2="281.94" y2="129.54" width="0.1524" layer="91"/>
-<wire x1="416.56" y1="119.38" x2="383.54" y2="119.38" width="0.1524" layer="91"/>
-<wire x1="383.54" y1="119.38" x2="373.38" y2="127" width="0.1524" layer="91"/>
+<wire x1="406.4" y1="149.86" x2="378.46" y2="127" width="0.1524" layer="91"/>
+<wire x1="378.46" y1="127" x2="373.38" y2="127" width="0.1524" layer="91"/>
 <label x="393.7" y="119.38" size="1.778" layer="95"/>
 <pinref part="TP2" gate="G$1" pin="1"/>
+<pinref part="X2" gate="G$1" pin="SWDIO"/>
+<wire x1="408.94" y1="147.32" x2="406.4" y2="149.86" width="0.1524" layer="91"/>
+<junction x="406.4" y="149.86"/>
 </segment>
 </net>
@@
 <label x="152.4" y="-15.24" size="1.778" layer="95"/>
 </segment>
+<segment>
+<pinref part="X2" gate="G$1" pin="VCC"/>
+<wire x1="424.18" y1="147.32" x2="426.72" y2="147.32" width="0.1524" layer="91"/>
+<label x="424.18" y="147.32" size="1.778" layer="95"/>
+</segment>
 </net>
 <net name="USB+" class="0">
@@
 <net name="SWCLK" class="0">
 <segment>
-<wire x1="416.56" y1="121.92" x2="383.54" y2="121.92" width="0.1524" layer="91"/>
+<wire x1="403.86" y1="149.86" x2="403.86" y2="144.78" width="0.1524" layer="91"/>
 <label x="393.7" y="121.92" size="1.778" layer="95"/>
-<wire x1="383.54" y1="121.92" x2="381" y2="124.46" width="0.1524" layer="91"/>
+<wire x1="403.86" y1="144.78" x2="381" y2="124.46" width="0.1524" layer="91"/>
 <wire x1="355.6" y1="124.46" x2="365.76" y2="124.46" width="0.1524" layer="91"/>
 <label x="373.38" y="124.46" size="1.778" layer="95" rot="MR0"/>
@@
 <wire x1="381" y1="124.46" x2="373.38" y2="124.46" width="0.1524" layer="91"/>
 <pinref part="TP1" gate="G$1" pin="1"/>
+<pinref part="X2" gate="G$1" pin="SWDCLK"/>
+<wire x1="408.94" y1="144.78" x2="403.86" y2="144.78" width="0.1524" layer="91"/>
+<junction x="403.86" y="144.78"/>
 </segment>
 </net>
@@
 <segment>
 <pinref part="R2" gate="G$1" pin="2"/>
-<wire x1="340.36" y1="144.78" x2="396.24" y2="144.78" width="0.1524" layer="91"/>
+<wire x1="340.36" y1="144.78" x2="391.16" y2="144.78" width="0.1524" layer="91"/>
+<wire x1="391.16" y1="144.78" x2="396.24" y2="144.78" width="0.1524" layer="91"/>
 <wire x1="396.24" y1="144.78" x2="396.24" y2="142.24" width="0.1524" layer="91"/>
 <label x="383.54" y="144.78" size="1.778" layer="95"/>
-</segment>
-</net>
+<pinref part="X2" gate="G$1" pin="NRESET"/>
+<wire x1="408.94" y1="137.16" x2="398.78" y2="137.16" width="0.1524" layer="91"/>
+<wire x1="398.78" y1="137.16" x2="391.16" y2="144.78" width="0.1524" layer="91"/>
+<junction x="391.16" y="144.78"/>
+</segment>
+</net>

Commit message: fully routed?
Parts:
- removed R9: 1K, microbuilder:RESISTOR_0603_NOOUT
- removed TP1, TP2: TEST-POINT3, SparkFun-Connectors:TEST-POINT3
- removed X2: 2x5 0.05" SWD, microbuilder:JTAG-CORTEXBOXPOSTS
- added R3: 1K, microbuilder:RESISTOR_0603_NOOUT
- added U$16: WINDBOND_QSPI_FLASHWSON_6X5, 00_bsiepert:WINDBOND_QSPI_FLASHWSON_6X5
- U$2: value WINDBOND_QSPI_FLASHUSON_2X3 -> SWD_HEADER; device 00_bsiepert:WINDBOND_QSPI_FLASHUSON_2X3 -> 00_bsiepert:SWD_HEADER
Connections:
- new net N$4: U$1.VDDCORE
- net GND: now also U$15.GND, U$16.GND, U$2.GND@1, U$2.GND@2, U$2.GND@3; no longer U$2.GND, X2.GND@1, X2.GND@2
- net QSPI_CS: now also U$16.CS; no longer U$2.CS
- net QSPI_IO0: now also U$16.DI/IO0; no longer U$2.DI/IO0
- net QSPI_IO1: now also U$16.DO/IO1; no longer U$2.DO/IO1
- net QSPI_IO2: now also U$16.WP/IO2; no longer U$2.WP/IO2
- net QSPI_IO3: now also U$16.HOLD/IO3; no longer U$2.HOLD/IO3
- net QSPI_SCK: now also U$16.CLK; no longer U$2.CLK
- net RESET_SW: now also U$2.RESET; no longer X2.NRESET
- net SWCLK: now also R3.1, U$2.SWDCLK; no longer R9.1, TP1.1, X2.SWDCLK
- net SWDIO: now also U$2.SWDIO; no longer TP2.1, X2.SWDIO
- net USB+: now also U$15.DATA+
- net USB-: now also U$15.DATA-
- net VDDCORE: no longer U$1.VDDCORE
- net VDDIO: now also R3.2, U$16.VCC; no longer R9.2, X2.VCC
Other:
- moved on the sheet: C1, R1, R2, SJ1

Commit message: mk1 fabbed
Parts:
- removed U$15: AMPHENOL_MICRO_USB, 00_bsiepert:AMPHENOL_MICRO_USB
- added U$19: AMPHENOL_MICRO_USBAMPHENOL_MICRO_USB_BETTER, 00_bsiepert:AMPHENOL_MICRO_USBAMPHENOL_MICRO_USB_BETTER
Connections:
- removed net N$4: U$1.VDDCORE
- net GND: now also U$19.GND; no longer U$15.GND
- net USB+: now also U$19.DATA+; no longer U$15.DATA+
- net USB-: now also U$19.DATA-; no longer U$15.DATA-
- net VDDCORE: now also U$1.VDDCORE
Changed lines of the file:
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@@
 <part name="U$14" library="microbuilder" deviceset="GND" device=""/>
 <part name="R2" library="microbuilder" deviceset="RESISTOR" device="_0603_NOOUT" value="330"/>
-<part name="U$15" library="00_bsiepert" deviceset="AMPHENOL_MICRO_USB" device=""/>
 <part name="U$16" library="00_bsiepert" deviceset="WINDBOND_QSPI_FLASH" device="WSON_6X5"/>
 <part name="U$2" library="00_bsiepert" deviceset="SWD_HEADER" device=""/>
@@
 <part name="R3" library="microbuilder" deviceset="RESISTOR" device="_0603_NOOUT" value="1K"/>
 <part name="U$18" library="microbuilder" deviceset="3.3V" device=""/>
+<part name="U$19" library="00_bsiepert" deviceset="AMPHENOL_MICRO_USB" device="AMPHENOL_MICRO_USB_BETTER"/>
 </parts>
 <sheets>
@@
 <instance part="U$14" gate="G$1" x="375.92" y="177.8" rot="R180"/>
 <instance part="R2" gate="G$1" x="381" y="193.04" rot="MR90"/>
-<instance part="U$15" gate="G$1" x="337.82" y="182.88" rot="R180"/>
 <instance part="U$16" gate="G$1" x="55.88" y="50.8"/>
 <instance part="U$2" gate="G$1" x="497.84" y="187.96" rot="R180"/>
@@
 <instance part="R3" gate="G$1" x="459.74" y="187.96" rot="MR90"/>
 <instance part="U$18" gate="G$1" x="528.32" y="182.88" rot="MR0"/>
+<instance part="U$19" gate="G$1" x="345.44" y="182.88" rot="R180"/>
 </instances>
 <busses>
@@
 </segment>
 <segment>
-<pinref part="U$15" gate="G$1" pin="GND"/>
 <wire x1="325.12" y1="193.04" x2="314.96" y2="193.04" width="0.1524" layer="91"/>
 <label x="317.5" y="193.04" size="1.778" layer="95"/>
+<pinref part="U$19" gate="G$1" pin="GND"/>
+<wire x1="332.74" y1="193.04" x2="325.12" y2="193.04" width="0.1524" layer="91"/>
 </segment>
 </net>
@@
 <wire x1="353.06" y1="93.98" x2="342.9" y2="93.98" width="0.1524" layer="91"/>
 <wire x1="342.9" y1="93.98" x2="337.82" y2="93.98" width="0.1524" layer="91"/>
-<wire x1="337.82" y1="93.98" x2="332.74" y2="99.06" width="0.1524" layer="91"/>
 <wire x1="342.9" y1="104.14" x2="342.9" y2="93.98" width="0.1524" layer="91"/>
 <junction x="342.9" y="93.98"/>
 <pinref part="C8" gate="G$1" pin="2"/>
+<pinref part="L1" gate="G$1" pin="2"/>
+<pinref part="U$1" gate="G$1" pin="VDDCORE"/>
+<wire x1="281.94" y1="104.14" x2="304.8" y2="104.14" width="0.1524" layer="91"/>
+<wire x1="304.8" y1="104.14" x2="312.42" y2="96.52" width="0.1524" layer="91"/>
+<wire x1="312.42" y1="96.52" x2="314.96" y2="93.98" width="0.1524" layer="91"/>
+<wire x1="314.96" y1="93.98" x2="337.82" y2="93.98" width="0.1524" layer="91"/>
 <junction x="337.82" y="93.98"/>
-<pinref part="L1" gate="G$1" pin="2"/>
-<wire x1="317.6524" y1="99.06" x2="332.74" y2="99.06" width="0.1524" layer="91"/>
 </segment>
 </net>
@@
 </segment>
 <segment>
-<pinref part="U$15" gate="G$1" pin="DATA-"/>
 <wire x1="325.12" y1="177.8" x2="314.96" y2="177.8" width="0.1524" layer="91"/>
 <label x="317.5" y="177.8" size="1.778" layer="95"/>
+<pinref part="U$19" gate="G$1" pin="DATA-"/>
+<wire x1="325.12" y1="177.8" x2="332.74" y2="177.8" width="0.1524" layer="91"/>
 </segment>
 </net>
@@
 </segment>
 <segment>
-<pinref part="U$15" gate="G$1" pin="DATA+"/>
 <wire x1="325.12" y1="182.88" x2="314.96" y2="182.88" width="0.1524" layer="91"/>
 <label x="317.5" y="182.88" size="1.778" layer="95"/>
+<pinref part="U$19" gate="G$1" pin="DATA+"/>
+<wire x1="325.12" y1="182.88" x2="332.74" y2="182.88" width="0.1524" layer="91"/>
 </segment>
 </net>
@@
 </segment>
 </net>
-<net name="N$4" class="0">
-<segment>
-<wire x1="309.88" y1="99.06" x2="317.3476" y2="99.06" width="0.1524" layer="91"/>
-<wire x1="304.8" y1="104.14" x2="309.88" y2="99.06" width="0.1524" layer="91"/>
-<pinref part="U$1" gate="G$1" pin="VDDCORE"/>
-<wire x1="281.94" y1="104.14" x2="304.8" y2="104.14" width="0.1524" layer="91"/>
-</segment>
-</net>
