File: cp32m4.sch (EAGLE design)
At the start: 19 parts, among them X5 32.768

Commit message: rename an updates
Connections:
- net GND: now also U$19.GND@1, U$19.GND@2, U$19.GND@3, U$19.GND@4
Other:
- moved on the sheet: C1
